Commit message: trying to make simulation easier

File: pybulletgym/envs/assets/robots/wolfgang/wolfgang_high_torque.urdf (robot description, URDF)
Before this commit: robot wolfgang, 26 links, 25 joints
Links:
- link l_foot: mass 0.312 -> 1; geometry collision box size=0.16 0.10 .04; visual box size=0.16 0.10 .04
- link r_foot: mass 0.312 -> 1; geometry collision box size=0.16 0.10 .04; visual box size=0.16 0.10 .04
